Commit message: refactor grasp planning and target ordering

File: grasp_core/resources/stand_v3.urf.xacro (robot description, xacro)
@@ -54,5 +54,5 @@
     <parent link="base_link"/>
     <child link="camera_rgb_link"/>
-    <origin rpy="-2.535527 -0.157327 -1.705899" xyz="0.195155 0.18463 1.305996"/>
+    <origin rpy="-2.535527 -0.157327 -1.705899" xyz="0.225155 0.18463 1.305996"/>
   </joint>
   <!-- <link name="camera_left_link"/>

Commit message: setup update

File: grasp_core/resources/stand_v3.urf.xacro (robot description, xacro)
@@ -54,5 +54,5 @@
     <parent link="base_link"/>
     <child link="camera_rgb_link"/>
-    <origin rpy="-2.535527 -0.157327 -1.705899" xyz="0.225155 0.18463 1.305996"/>
+    <origin rpy="-2.736556 -0.006884 -1.598774" xyz="0.099802 0.037719 1.227970"/>
   </joint>
   <!-- <link name="camera_left_link"/>
